File: cici.sch (KiCad schematic (older format))
At the start: 43 parts, among them SW1 SW_PUSH, SW10 SW_PUSH, SW11 SW_PUSH, SW12 SW_PUSH, SW13 SW_PUSH, SW14 SW_PUSH, SW15 SW_PUSH, SW16 SW_PUSH, SW17 SW_PUSH, SW18 SW_PUSH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

Commit message: update
Parts:
- removed LED1, LED2: POWER, LED_THT:LED_D3.0mm, symbol Device:LED
- removed R1, R2: 1.5K, Resistor_THT:R_Axial_DIN0204_L3.6mm_D1.6mm_P7.62mm_Horizontal, symbol Device:R_Small
- removed RSW1: SW_PUSH, kbd:ResetSW_1side, symbol cici-rescue:SW_PUSH-kbd-corne-light-rescue
- added SW_R: SW_PUSH, kbd:ResetSW_1side, symbol kbd:SW_PUSH
- renumbered OLED to OLED1
Connections:
- net labels removed: +5V, VDD
Changed lines of the file:
@@
-	1    0    0    -1
-$EndComp
-$Comp
-L cici-rescue:SW_PUSH-kbd-corne-light-rescue RSW1
-U 1 1 625312FA
-P 8700 2275
-F 0 "RSW1" H 8700 2530 50  0000 C CNN
-F 1 "SW_PUSH" H 8700 2439 50  0000 C CNN
-F 2 "kbd:ResetSW_1side" H 8700 2275 50  0001 C CNN
-F 3 "" H 8700 2275 50  0000 C CNN
-	1    8700 2275
 	1    0    0    -1
 $EndComp
@@
 Wire Wire Line
 	5450 2675 5550 2675
-$Comp
-L Device:LED LED1
-U 1 1 625207E7
-P 8800 2775
-F 0 "LED1" H 8793 2900 50  0000 C CNN
-F 1 "POWER" H 8793 2900 50  0001 C CNN
-F 2 "LED_THT:LED_D3.0mm" H 8800 2775 50  0001 C CNN
-F 3 "~" H 8800 2775 50  0001 C CNN
-	1    8800 2775
-	1    0    0    -1
-$EndComp
-$Comp
-L power:+5V #PWR0114
-U 1 1 62522850
-P 8950 2775
-F 0 "#PWR0114" H 8950 2625 50  0001 C CNN
-F 1 "+5V" H 8965 2948 50  0000 C CNN
-F 2 "" H 8950 2775 50  0001 C CNN
-F 3 "" H 8950 2775 50  0001 C CNN
-	1    8950 2775
-	1    0    0    -1
-$EndComp
-$Comp
-L Device:R_Small R1
-U 1 1 62524923
-P 8550 2775
-F 0 "R1" V 8354 2775 50  0000 C CNN
-F 1 "1.5K" V 8445 2775 50  0000 C CNN
-F 2 "Resistor_THT:R_Axial_DIN0204_L3.6mm_D1.6mm_P7.62mm_Horizontal" H 8550 2775 50  0001 C CNN
-F 3 "~" H 8550 2775 50  0001 C CNN
-	1    8550 2775
-	0    1    1    0
-$EndComp
-$Comp
-L power:GND #PWR0113
-U 1 1 62523C57
-P 8450 2775
-F 0 "#PWR0113" H 8450 2525 50  0001 C CNN
-F 1 "GND" H 8455 2602 50  0000 C CNN
-F 2 "" H 8450 2775 50  0001 C CNN
-F 3 "" H 8450 2775 50  0001 C CNN
-	1    8450 2775
-	1    0    0    -1
-$EndComp
 Text GLabel 5625 3375 0    50   Input ~ 0
 row4
@@
 Connection ~ 1200 4550
 Connection ~ 1925 4550
-$Comp
-L Device:LED LED2
-U 1 1 625CA200
-P 8800 3275
-F 0 "LED2" H 8793 3400 50  0000 C CNN
-F 1 "POWER" H 8793 3400 50  0001 C CNN
-F 2 "LED_THT:LED_D3.0mm" H 8800 3275 50  0001 C CNN
-F 3 "~" H 8800 3275 50  0001 C CNN
-	1    8800 3275
-	1    0    0    -1
-$EndComp
-$Comp
-L Device:R_Small R2
-U 1 1 625CA798
-P 8550 3275
-F 0 "R2" V 8354 3275 50  0000 C CNN
-F 1 "1.5K" V 8445 3275 50  0000 C CNN
-F 2 "Resistor_THT:R_Axial_DIN0204_L3.6mm_D1.6mm_P7.62mm_Horizontal" H 8550 3275 50  0001 C CNN
-F 3 "~" H 8550 3275 50  0001 C CNN
-	1    8550 3275
-	0    1    1    0
-$EndComp
-$Comp
-L power:GND #PWR?
-U 1 1 625CAD49
-P 8450 3275
-F 0 "#PWR?" H 8450 3025 50  0001 C CNN
-F 1 "GND" H 8455 3102 50  0000 C CNN
-F 2 "" H 8450 3275 50  0001 C CNN
-F 3 "" H 8450 3275 50  0001 C CNN
-	1    8450 3275
-	1    0    0    -1
-$EndComp
-$Comp
-L power:+5V #PWR?
-U 1 1 625CB500
-P 8950 3275
-F 0 "#PWR?" H 8950 3125 50  0001 C CNN
-F 1 "+5V" H 8965 3448 50  0000 C CNN
-F 2 "" H 8950 3275 50  0001 C CNN
-F 3 "" H 8950 3275 50  0001 C CNN
-	1    8950 3275
-	1    0    0    -1
-$EndComp
 Wire Wire Line
 	2775 2175 2775 2525
@@
 $EndComp
 $Comp
-L kbd:OLED OLED
+L kbd:OLED OLED1
 U 1 1 62546E3D
 P 6125 4500
-F 0 "OLED" H 6753 4525 51  0000 L CNN
+F 0 "OLED1" H 6753 4525 51  0000 L CNN
 F 1 "OLED" H 6753 4479 47  0001 L CNN
 F 2 "kbd:OLED_1side" H 6125 4600 60  0001 C CNN
@@
 Connection ~ 2050 2525
 $Comp
-L power:VDD #PWR?
-U 1 1 62541D3A
-P 5375 4550
-F 0 "#PWR?" H 5375 4400 50  0001 C CNN
-F 1 "VDD" V 5393 4677 50  0000 L CNN
-F 2 "" H 5375 4550 50  0001 C CNN
-F 3 "" H 5375 4550 50  0001 C CNN
-	1    5375 4550
-	0    -1   -1   0
-$EndComp
-$Comp
-L power:GND #PWR?
+L power:GND #PWR0104
 U 1 1 62542DB1
 P 5375 4700
-F 0 "#PWR?" H 5375 4450 50  0001 C CNN
+F 0 "#PWR0104" H 5375 4450 50  0001 C CNN
 F 1 "GND" V 5380 4572 50  0000 R CNN
 F 2 "" H 5375 4700 50  0001 C CNN
@@
 Text GLabel 5375 4250 0    50   Input ~ 0
 SDA
+$Comp
+L power:VCC #PWR0101
+U 1 1 6254B58B
+P 5375 4550
+F 0 "#PWR0101" H 5375 4400 50  0001 C CNN
+F 1 "VCC" V 5393 4677 50  0000 L CNN
+F 2 "" H 5375 4550 50  0001 C CNN
+F 3 "" H 5375 4550 50  0001 C CNN
+	1    5375 4550
+	0    -1   -1   0
+$EndComp
+$Comp
+L kbd:SW_PUSH SW_R
+U 1 1 6254F34F
+P 8700 2275
+F 0 "SW_R" H 8700 2438 50  0000 C CNN
+F 1 "SW_PUSH" H 8700 2529 50  0001 C CNN
+F 2 "kbd:ResetSW_1side" H 8700 2438 50  0001 C CNN
+F 3 "" H 8700 2275 50  0000 C CNN
+	1    8700 2275
+	1    0    0    -1
+$EndComp
 $EndSCHEMATC

Commit message: realizzato bottom e sistemato fori per viti
Parts:
- renumbered SW_R to SW_R1
Changed lines of the file:
@@
 $EndComp
 $Comp
-L kbd:SW_PUSH SW_R
+L kbd:SW_PUSH SW_R1
 U 1 1 6254F34F
 P 8700 2275
-F 0 "SW_R" H 8700 2438 50  0000 C CNN
+F 0 "SW_R1" H 8700 2438 50  0000 C CNN
 F 1 "SW_PUSH" H 8700 2529 50  0001 C CNN
 F 2 "kbd:ResetSW_1side" H 8700 2438 50  0001 C CNN

Commit message: prima versione conclusa. inizio seconda
Parts:
- added H? (x8): MountingHole, MountingHole:MountingHole_2.2mm_M2_Pad, symbol Mechanical:MountingHole
- SW1, SW10, SW11, SW12, SW13, SW14, SW15, SW16, SW17, SW18, SW2, SW3, SW4, SW5, SW6, SW7, SW8, SW9: footprint kbd:keyswitch_cherrymx_alps_choc12_1u -> kbd:CherryMX_1u
Changed lines of the file:
@@
 F 0 "SW1" H 900 2688 50  0000 C CNN
 F 1 "SW_PUSH" H 900 2689 50  0001 C CNN
-F 2 "kbd:keyswitch_cherrymx_alps_choc12_1u" H 900 2525 50  0001 C CNN
+F 2 "kbd:CherryMX_1u" H 900 2525 50  0001 C CNN
 F 3 "" H 900 2525 50  0000 C CNN
 	1    900  2525
@@
 F 0 "SW2" H 1625 2688 50  0000 C CNN
 F 1 "SW_PUSH" H 1625 2689 50  0001 C CNN
-F 2 "kbd:keyswitch_cherrymx_alps_choc12_1u" H 1625 2525 50  0001 C CNN
+F 2 "kbd:CherryMX_1u" H 1625 2525 50  0001 C CNN
 F 3 "" H 1625 2525 50  0000 C CNN
 	1    1625 2525
@@
 F 0 "SW6" H 1625 3355 50  0000 C CNN
 F 1 "SW_PUSH" H 1625 3264 50  0001 C CNN
-F 2 "kbd:keyswitch_cherrymx_alps_choc12_1u" H 1625 3100 50  0001 C CNN
+F 2 "kbd:CherryMX_1u" H 1625 3100 50  0001 C CNN
 F 3 "" H 1625 3100 50  0000 C CNN
 	1    1625 3100
@@
 F 0 "SW5" H 900 3263 50  0000 C CNN
 F 1 "SW_PUSH" H 900 3264 50  0001 C CNN
-F 2 "kbd:keyswitch_cherrymx_alps_choc12_1u" H 900 3100 50  0001 C CNN
+F 2 "kbd:CherryMX_1u" H 900 3100 50  0001 C CNN
 F 3 "" H 900 3100 50  0000 C CNN
 	1    900  3100
@@
 F 0 "SW3" H 2350 2688 50  0000 C CNN
 F 1 "SW_PUSH" H 2350 2689 50  0001 C CNN
-F 2 "kbd:keyswitch_cherrymx_alps_choc12_1u" H 2350 2525 50  0001 C CNN
+F 2 "kbd:CherryMX_1u" H 2350 2525 50  0001 C CNN
 F 3 "" H 2350 2525 50  0000 C CNN
 	1    2350 2525
@@
 F 0 "SW4" H 3075 2688 50  0000 C CNN
 F 1 "SW_PUSH" H 3075 2689 50  0001 C CNN
-F 2 "kbd:keyswitch_cherrymx_alps_choc12_1u" H 3075 2525 50  0001 C CNN
+F 2 "kbd:CherryMX_1u" H 3075 2525 50  0001 C CNN
 F 3 "" H 3075 2525 50  0000 C CNN
 	1    3075 2525
@@
 F 0 "SW9" H 900 3930 50  0000 C CNN
 F 1 "SW_PUSH" H 900 3839 50  0001 C CNN
-F 2 "kbd:keyswitch_cherrymx_alps_choc12_1u" H 900 3675 50  0001 C CNN
+F 2 "kbd:CherryMX_1u" H 900 3675 50  0001 C CNN
 F 3 "" H 900 3675 50  0000 C CNN
 	1    900  3675
@@
 F 0 "SW18" H 2350 4988 50  0000 C CNN
 F 1 "SW_PUSH" H 2350 4989 50  0001 C CNN
-F 2 "kbd:keyswitch_cherrymx_alps_choc12_1u" H 2350 4825 50  0001 C CNN
+F 2 "kbd:CherryMX_1u" H 2350 4825 50  0001 C CNN
 F 3 "" H 2350 4825 50  0000 C CNN
 	1    2350 4825
@@
 F 0 "SW17" H 1625 4988 50  0000 C CNN
 F 1 "SW_PUSH" H 1625 4989 50  0001 C CNN
-F 2 "kbd:keyswitch_cherrymx_alps_choc12_1u" H 1625 4825 50  0001 C CNN
+F 2 "kbd:CherryMX_1u" H 1625 4825 50  0001 C CNN
 F 3 "" H 1625 4825 50  0000 C CNN
 	1    1625 4825
@@
 F 0 "SW13" H 900 4413 50  0000 C CNN
 F 1 "SW_PUSH" H 900 4414 50  0001 C CNN
-F 2 "kbd:keyswitch_cherrymx_alps_choc12_1u" H 900 4250 50  0001 C CNN
+F 2 "kbd:CherryMX_1u" H 900 4250 50  0001 C CNN
 F 3 "" H 900 4250 50  0000 C CNN
 	1    900  4250
@@
 F 0 "SW10" H 1625 3930 50  0000 C CNN
 F 1 "SW_PUSH" H 1625 3839 50  0001 C CNN
-F 2 "kbd:keyswitch_cherrymx_alps_choc12_1u" H 1625 3675 50  0001 C CNN
+F 2 "kbd:CherryMX_1u" H 1625 3675 50  0001 C CNN
 F 3 "" H 1625 3675 50  0000 C CNN
 	1    1625 3675
@@
 F 0 "SW14" H 1625 4413 50  0000 C CNN
 F 1 "SW_PUSH" H 1625 4414 50  0001 C CNN
-F 2 "kbd:keyswitch_cherrymx_alps_choc12_1u" H 1625 4250 50  0001 C CNN
+F 2 "kbd:CherryMX_1u" H 1625 4250 50  0001 C CNN
 F 3 "" H 1625 4250 50  0000 C CNN
 	1    1625 4250
@@
 F 0 "SW15" H 2350 4413 50  0000 C CNN
 F 1 "SW_PUSH" H 2350 4414 50  0001 C CNN
-F 2 "kbd:keyswitch_cherrymx_alps_choc12_1u" H 2350 4250 50  0001 C CNN
+F 2 "kbd:CherryMX_1u" H 2350 4250 50  0001 C CNN
 F 3 "" H 2350 4250 50  0000 C CNN
 	1    2350 4250
@@
 F 0 "SW16" H 3075 4413 50  0000 C CNN
 F 1 "SW_PUSH" H 3075 4414 50  0001 C CNN
-F 2 "kbd:keyswitch_cherrymx_alps_choc12_1u" H 3075 4250 50  0001 C CNN
+F 2 "kbd:CherryMX_1u" H 3075 4250 50  0001 C CNN
 F 3 "" H 3075 4250 50  0000 C CNN
 	1    3075 4250
@@
 F 0 "SW12" H 3075 3930 50  0000 C CNN
 F 1 "SW_PUSH" H 3075 3839 50  0001 C CNN
-F 2 "kbd:keyswitch_cherrymx_alps_choc12_1u" H 3075 3675 50  0001 C CNN
+F 2 "kbd:CherryMX_1u" H 3075 3675 50  0001 C CNN
 F 3 "" H 3075 3675 50  0000 C CNN
 	1    3075 3675
@@
 F 0 "SW11" H 2350 3930 50  0000 C CNN
 F 1 "SW_PUSH" H 2350 3839 50  0001 C CNN
-F 2 "kbd:keyswitch_cherrymx_alps_choc12_1u" H 2350 3675 50  0001 C CNN
+F 2 "kbd:CherryMX_1u" H 2350 3675 50  0001 C CNN
 F 3 "" H 2350 3675 50  0000 C CNN
 	1    2350 3675
@@
 F 0 "SW7" H 2350 3355 50  0000 C CNN
 F 1 "SW_PUSH" H 2350 3264 50  0001 C CNN
-F 2 "kbd:keyswitch_cherrymx_alps_choc12_1u" H 2350 3100 50  0001 C CNN
+F 2 "kbd:CherryMX_1u" H 2350 3100 50  0001 C CNN
 F 3 "" H 2350 3100 50  0000 C CNN
 	1    2350 3100
@@
 F 0 "SW8" H 3075 3355 50  0000 C CNN
 F 1 "SW_PUSH" H 3075 3264 50  0001 C CNN
-F 2 "kbd:keyswitch_cherrymx_alps_choc12_1u" H 3075 3100 50  0001 C CNN
+F 2 "kbd:CherryMX_1u" H 3075 3100 50  0001 C CNN
 F 3 "" H 3075 3100 50  0000 C CNN
 	1    3075 3100
@@
 	1    0    0    -1
 $EndComp
+$Comp
+L Mechanical:MountingHole H?
+U 1 1 626C7888
+P 4375 2750
+F 0 "H?" H 4475 2796 50  0001 L CNN
+F 1 "MountingHole" H 4475 2750 50  0000 L CNN
+F 2 "MountingHole:MountingHole_2.2mm_M2_Pad" H 4375 2750 50  0001 C CNN
+F 3 "~" H 4375 2750 50  0001 C CNN
+	1    4375 2750
+	1    0    0    -1
+$EndComp
+$Comp
+L Mechanical:MountingHole H?
+U 1 1 626C9167
+P 4375 3000
+F 0 "H?" H 4475 3046 50  0001 L CNN
+F 1 "MountingHole" H 4475 3000 50  0000 L CNN
+F 2 "MountingHole:MountingHole_2.2mm_M2_Pad" H 4375 3000 50  0001 C CNN
+F 3 "~" H 4375 3000 50  0001 C CNN
+	1    4375 3000
+	1    0    0    -1
+$EndComp
+$Comp
+L Mechanical:MountingHole H?
+U 1 1 626C99B8
+P 4375 3250
+F 0 "H?" H 4475 3296 50  0001 L CNN
+F 1 "MountingHole" H 4475 3250 50  0000 L CNN
+F 2 "MountingHole:MountingHole_2.2mm_M2_Pad" H 4375 3250 50  0001 C CNN
+F 3 "~" H 4375 3250 50  0001 C CNN
+	1    4375 3250
+	1    0    0    -1
+$EndComp
+$Comp
+L Mechanical:MountingHole H?
+U 1 1 626C9BC6
+P 4375 3500
+F 0 "H?" H 4475 3546 50  0001 L CNN
+F 1 "MountingHole" H 4475 3500 50  0000 L CNN
+F 2 "MountingHole:MountingHole_2.2mm_M2_Pad" H 4375 3500 50  0001 C CNN
+F 3 "~" H 4375 3500 50  0001 C CNN
+	1    4375 3500
+	1    0    0    -1
+$EndComp
+$Comp
+L Mechanical:MountingHole H?
+U 1 1 626C9E42
+P 4375 3750
+F 0 "H?" H 4475 3796 50  0001 L CNN
+F 1 "MountingHole" H 4475 3750 50  0000 L CNN
+F 2 "MountingHole:MountingHole_2.2mm_M2_Pad" H 4375 3750 50  0001 C CNN
+F 3 "~" H 4375 3750 50  0001 C CNN
+	1    4375 3750
+	1    0    0    -1
+$EndComp
+$Comp
+L Mechanical:MountingHole H?
+U 1 1 626CA15D
+P 4375 4000
+F 0 "H?" H 4475 4046 50  0001 L CNN
+F 1 "MountingHole" H 4475 4000 50  0000 L CNN
+F 2 "MountingHole:MountingHole_2.2mm_M2_Pad" H 4375 4000 50  0001 C CNN
+F 3 "~" H 4375 4000 50  0001 C CNN
+	1    4375 4000
+	1    0    0    -1
+$EndComp
+$Comp
+L Mechanical:MountingHole H?
+U 1 1 626CA45B
+P 4375 4250
+F 0 "H?" H 4475 4296 50  0001 L CNN
+F 1 "MountingHole" H 4475 4250 50  0000 L CNN
+F 2 "MountingHole:MountingHole_2.2mm_M2_Pad" H 4375 4250 50  0001 C CNN
+F 3 "~" H 4375 4250 50  0001 C CNN
+	1    4375 4250
+	1    0    0    -1
+$EndComp
+$Comp
+L Mechanical:MountingHole H?
+U 1 1 626CA6AA
+P 4375 4500
+F 0 "H?" H 4475 4546 50  0001 L CNN
+F 1 "MountingHole" H 4475 4500 50  0000 L CNN
+F 2 "MountingHole:MountingHole_2.2mm_M2_Pad" H 4375 4500 50  0001 C CNN
+F 3 "~" H 4375 4500 50  0001 C CNN
+	1    4375 4500
+	1    0    0    -1
+$EndComp
