File: cici_pcb/cici.kicad_pcb (KiCad board)
At the start: 2 copper layers, 88.4 x 140.3 mm, 47 parts, among them SW1 SW_PUSH, SW10 SW_PUSH, SW11 SW_PUSH, SW12 SW_PUSH, SW13 SW_PUSH, SW14 SW_PUSH, SW15 SW_PUSH, SW16 SW_PUSH, SW17 SW_PUSH, SW18 SW_PUSH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

Commit message: aggiornamento pcb
Parts:
- D1, D10, D11, D12, D13, D14, D15, D16, D17, D18, D2, D3, D4, D5, D6, D7, D8, D9: footprint kbd:D3_TH -> cftkb:D_DO-35_SOD27_P5.08mm_Horizontal
- moved D10 4.95 mm to (103.1, 46.4)
- moved D11 4.95 mm to (106.1, 46.4)
- moved D12 4.95 mm to (109.1, 46.4)
- moved D13 4.95 mm to (112.1, 46.4)
- moved D14 4.95 mm to (115.1, 46.4)
- moved D15 4.95 mm to (118.1, 46.4)
- moved D16 4.95 mm to (121.1, 46.4)
- moved D17 4.95 mm to (124.1, 46.4)
- moved D18 4.95 mm to (127.1, 46.4)
- moved D1 4.60 mm to (103.1, 34.7)
- moved D2 4.60 mm to (106.1, 34.7)
- moved D3 4.60 mm to (109.1, 34.7)
- moved D4 4.60 mm to (112.1, 34.7)
- moved D5 4.60 mm to (115.1, 34.7)
- moved D6 4.60 mm to (118.1, 34.7)
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Routing:
- net Net-(D9-Pad2): track 153.2 -> 139.1 mm, vias 2 -> 1
- net row1: track 75.4 -> 67.8 mm, vias 1 -> 0
- net Net-(D12-Pad2): track 86.9 -> 81.2 mm, vias 2 -> 1
- net Net-(D11-Pad2): track 108.2 -> 102.6 mm, vias 2 -> 1
- net row2: track 112.8 -> 107.4 mm, vias 1 -> 0
- net Net-(D13-Pad2): track 162.2 -> 156.8 mm, vias 2 -> 1
- net Net-(D10-Pad2): track 126.8 -> 121.7 mm, vias 2 -> 1
- net Net-(D16-Pad2): track 95.3 -> 90.7 mm, vias 2 -> 1
- net Net-(D14-Pad2): track 141.3 -> 136.7 mm, vias 2 -> 1
- net Net-(D15-Pad2): track 118.0 -> 113.6 mm, vias 2 -> 1
- net row4: track 78.5 -> 82.2 mm, vias 3 -> 2
- net Net-(D18-Pad2): track 122.7 -> 119.6 mm, vias 0 -> 1
- net row0: track 60.2 -> 57.4 mm, vias 1 -> 0
- net VCC: track 28.4 -> 31.1 mm
- net Net-(D4-Pad2): track 70.9 -> 68.9 mm, vias 2 -> 1
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