File: cici_pcb/cici.sch (KiCad schematic (older format))
At the start: 47 parts, among them SW1 SW_PUSH, SW10 SW_PUSH, SW11 SW_PUSH, SW12 SW_PUSH, SW13 SW_PUSH, SW14 SW_PUSH, SW15 SW_PUSH, SW16 SW_PUSH, SW17 SW_PUSH, SW18 SW_PUSH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

Commit message: aggiornamento pcb
Parts:
- D1, D10, D11, D12, D13, D14, D15, D16, D17, D18, D2, D3, D4, D5, D6, D7, D8, D9: footprint kbd:D3_TH -> cftkb:D_DO-35_SOD27_P5.08mm_Horizontal
Changed lines of the file:
@@
 F 0 "D1" V 1246 2596 50  0000 R CNN
 F 1 "D" V 1155 2596 50  0001 R CNN
-F 2 "kbd:D3_TH" H 1200 2675 50  0001 C CNN
+F 2 "cftkb:D_DO-35_SOD27_P5.08mm_Horizontal" H 1200 2675 50  0001 C CNN
 F 3 "~" H 1200 2675 50  0001 C CNN
 	1    1200 2675
@@
 F 0 "D2" V 1971 2596 50  0000 R CNN
 F 1 "D" V 1880 2596 50  0001 R CNN
-F 2 "kbd:D3_TH" H 1925 2675 50  0001 C CNN
+F 2 "cftkb:D_DO-35_SOD27_P5.08mm_Horizontal" H 1925 2675 50  0001 C CNN
 F 3 "~" H 1925 2675 50  0001 C CNN
 	1    1925 2675
@@
 F 0 "D3" V 2696 2596 50  0000 R CNN
 F 1 "D" V 2605 2596 50  0001 R CNN
-F 2 "kbd:D3_TH" H 2650 2675 50  0001 C CNN
+F 2 "cftkb:D_DO-35_SOD27_P5.08mm_Horizontal" H 2650 2675 50  0001 C CNN
 F 3 "~" H 2650 2675 50  0001 C CNN
 	1    2650 2675
@@
 F 0 "D4" V 3421 2596 50  0000 R CNN
 F 1 "D" V 3330 2596 50  0001 R CNN
-F 2 "kbd:D3_TH" H 3375 2675 50  0001 C CNN
+F 2 "cftkb:D_DO-35_SOD27_P5.08mm_Horizontal" H 3375 2675 50  0001 C CNN
 F 3 "~" H 3375 2675 50  0001 C CNN
 	1    3375 2675
@@
 F 0 "D5" V 1246 3171 50  0000 R CNN
 F 1 "D" V 1155 3171 50  0001 R CNN
-F 2 "kbd:D3_TH" H 1200 3250 50  0001 C CNN
+F 2 "cftkb:D_DO-35_SOD27_P5.08mm_Horizontal" H 1200 3250 50  0001 C CNN
 F 3 "~" H 1200 3250 50  0001 C CNN
 	1    1200 3250
@@
 F 0 "D9" V 1246 3746 50  0000 R CNN
 F 1 "D" V 1155 3746 50  0001 R CNN
-F 2 "kbd:D3_TH" H 1200 3825 50  0001 C CNN
+F 2 "cftkb:D_DO-35_SOD27_P5.08mm_Horizontal" H 1200 3825 50  0001 C CNN
 F 3 "~" H 1200 3825 50  0001 C CNN
 	1    1200 3825
@@
 F 0 "D10" V 1971 3746 50  0000 R CNN
 F 1 "D" V 1880 3746 50  0001 R CNN
-F 2 "kbd:D3_TH" H 1925 3825 50  0001 C CNN
+F 2 "cftkb:D_DO-35_SOD27_P5.08mm_Horizontal" H 1925 3825 50  0001 C CNN
 F 3 "~" H 1925 3825 50  0001 C CNN
 	1    1925 3825
@@
 F 0 "D6" V 1971 3171 50  0000 R CNN
 F 1 "D" V 1880 3171 50  0001 R CNN
-F 2 "kbd:D3_TH" H 1925 3250 50  0001 C CNN
+F 2 "cftkb:D_DO-35_SOD27_P5.08mm_Horizontal" H 1925 3250 50  0001 C CNN
 F 3 "~" H 1925 3250 50  0001 C CNN
 	1    1925 3250
@@
 F 0 "D7" V 2696 3171 50  0000 R CNN
 F 1 "D" V 2605 3171 50  0001 R CNN
-F 2 "kbd:D3_TH" H 2650 3250 50  0001 C CNN
+F 2 "cftkb:D_DO-35_SOD27_P5.08mm_Horizontal" H 2650 3250 50  0001 C CNN
 F 3 "~" H 2650 3250 50  0001 C CNN
 	1    2650 3250
@@
 F 0 "D8" V 3421 3171 50  0000 R CNN
 F 1 "D" V 3330 3171 50  0001 R CNN
-F 2 "kbd:D3_TH" H 3375 3250 50  0001 C CNN
+F 2 "cftkb:D_DO-35_SOD27_P5.08mm_Horizontal" H 3375 3250 50  0001 C CNN
 F 3 "~" H 3375 3250 50  0001 C CNN
 	1    3375 3250
@@
 F 0 "D17" V 1971 4896 50  0000 R CNN
 F 1 "D" V 1880 4896 50  0001 R CNN
-F 2 "kbd:D3_TH" H 1925 4975 50  0001 C CNN
+F 2 "cftkb:D_DO-35_SOD27_P5.08mm_Horizontal" H 1925 4975 50  0001 C CNN
 F 3 "~" H 1925 4975 50  0001 C CNN
 	1    1925 4975
@@
 F 0 "D18" V 2696 4896 50  0000 R CNN
 F 1 "D" V 2605 4896 50  0001 R CNN
-F 2 "kbd:D3_TH" H 2650 4975 50  0001 C CNN
+F 2 "cftkb:D_DO-35_SOD27_P5.08mm_Horizontal" H 2650 4975 50  0001 C CNN
 F 3 "~" H 2650 4975 50  0001 C CNN
 	1    2650 4975
@@
 F 0 "D16" V 3421 4321 50  0000 R CNN
 F 1 "D" V 3330 4321 50  0001 R CNN
-F 2 "kbd:D3_TH" H 3375 4400 50  0001 C CNN
+F 2 "cftkb:D_DO-35_SOD27_P5.08mm_Horizontal" H 3375 4400 50  0001 C CNN
 F 3 "~" H 3375 4400 50  0001 C CNN
 	1    3375 4400
@@
 F 0 "D14" V 1971 4321 50  0000 R CNN
 F 1 "D" V 1880 4321 50  0001 R CNN
-F 2 "kbd:D3_TH" H 1925 4400 50  0001 C CNN
+F 2 "cftkb:D_DO-35_SOD27_P5.08mm_Horizontal" H 1925 4400 50  0001 C CNN
 F 3 "~" H 1925 4400 50  0001 C CNN
 	1    1925 4400
@@
 F 0 "D13" V 1246 4321 50  0000 R CNN
 F 1 "D" V 1155 4321 50  0001 R CNN
-F 2 "kbd:D3_TH" H 1200 4400 50  0001 C CNN
+F 2 "cftkb:D_DO-35_SOD27_P5.08mm_Horizontal" H 1200 4400 50  0001 C CNN
 F 3 "~" H 1200 4400 50  0001 C CNN
 	1    1200 4400
@@
 F 0 "D11" V 2696 3746 50  0000 R CNN
 F 1 "D" V 2605 3746 50  0001 R CNN
-F 2 "kbd:D3_TH" H 2650 3825 50  0001 C CNN
+F 2 "cftkb:D_DO-35_SOD27_P5.08mm_Horizontal" H 2650 3825 50  0001 C CNN
 F 3 "~" H 2650 3825 50  0001 C CNN
 	1    2650 3825
@@
 F 0 "D12" V 3421 3746 50  0000 R CNN
 F 1 "D" V 3330 3746 50  0001 R CNN
-F 2 "kbd:D3_TH" H 3375 3825 50  0001 C CNN
+F 2 "cftkb:D_DO-35_SOD27_P5.08mm_Horizontal" H 3375 3825 50  0001 C CNN
 F 3 "~" H 3375 3825 50  0001 C CNN
 	1    3375 3825
@@
 F 0 "D15" V 2696 4321 50  0000 R CNN
 F 1 "D" V 2605 4321 50  0001 R CNN
-F 2 "kbd:D3_TH" H 2650 4400 50  0001 C CNN
+F 2 "cftkb:D_DO-35_SOD27_P5.08mm_Horizontal" H 2650 4400 50  0001 C CNN
 F 3 "~" H 2650 4400 50  0001 C CNN
 	1    2650 4400
